File: modifiedradio.sch (EAGLE design)
At the start: 18 parts, among them IC1 74164D

Commit message: added schematic
Connections:
- net GND: now also DIS1.R/W
Changed lines of the file:
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@@
 <part name="P+4" library="supply1" deviceset="+5V" device=""/>
 <part name="GND9" library="supply1" deviceset="GND" device=""/>
+<part name="GND10" library="supply1" deviceset="GND" device=""/>
 </parts>
 <sheets>
@@
 <instance part="P+4" gate="1" x="76.2" y="99.06"/>
 <instance part="GND9" gate="1" x="83.82" y="101.6"/>
+<instance part="GND10" gate="1" x="-17.78" y="33.02"/>
 </instances>
 <busses>
@@
 <label x="38.1" y="71.12" size="1.778" layer="95"/>
 </segment>
+<segment>
+<pinref part="DIS1" gate="G$1" pin="R/W"/>
+<pinref part="GND10" gate="1" pin="GND"/>
+<wire x1="-17.78" y1="48.26" x2="-17.78" y2="35.56" width="0.1524" layer="91"/>
+</segment>
 </net>
